File: SE30-Grayscale.kicad_pcb (KiCad board)
At the start: 2 copper layers, 85.7 x 69.8 mm, 31 parts, among them J1 Molex, 8P RA, Q1 2N5550TFR, Q2 2N5550TFR, Q3 PN2222A

Commit message: Updated tube socket footprint
This matches the specification listed on the Pacific TV website for the 7-pin miniature tube socket they sell; the old footprint probably would have fit fine, since it was close, but why risk it?
Parts:
- V1: footprint SE30-Grayscale:Tube_7pin_Mini -> SE30-Grayscale:Tube_Socket_China
